File: Solenoid_UNIT.kicad_pcb (KiCad board)
At the start: 2 copper layers, 20.6 x 28 mm, 11 parts, among them CN1 CON_GROVE, J2 Conn_01x04, Q1 TR_nMOS_IRF7103

Commit message: add images
Parts:
- moved JP1 6.49 mm to (13.0, 12.0), turned to -90 degrees
- moved JP2 3.01 mm to (9.50, 12.0), turned to -90 degrees
Connections:
- J2 pad 1: /SOLA_M -> GND
- J2 pad 2: /SOLA_P2 -> VDD
- J2 pad 3: VDD -> /SOLA_P2
- J2 pad 4: GND -> /SOLA_M
Routing:
- net GND: track 34.4 -> 53.3 mm
- net Net-(Q1-Pad4): track 30.7 -> 13.3 mm
- net /SOLA_M: track 7.58 -> 14.4 mm
- net VS: track 19.1 -> 13.8 mm
- net /SOLA_P2: track 3.68 -> 8.09 mm
- net /SOLB_M: track 9.23 -> 6.42 mm, vias 2 -> 1
- net VDD: track 5.59 -> 3.90 mm
- net +5V: track 12.8 -> 13.6 mm
- net Net-(Q1-Pad2): track 20.1 -> 19.4 mm
Other:
- board text added: "Grove"
- board text added: "useB"
