File: Solenoid_UNIT.kicad_sch (KiCad schematic)
At the start: 11 parts, among them CN1 CON_GROVE, J2 Conn_01x04, Q1 TR_nMOS_IRF7103

Commit message: add images
Connections:
- net GND: now also J2.1 (Pin_1); no longer J2.4 (Pin_4)
- net SOLA_M: now also J2.4 (Pin_4); no longer J2.1 (Pin_1)
- net SOLA_P2: now also J2.3 (Pin_3); no longer J2.2 (Pin_2)
- net VDD: now also J2.2 (Pin_2); no longer J2.3 (Pin_3)
Changed lines of the file:
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@@
     (pin "1")
   )
-  (symbol (lib_id "Connector_Generic:Conn_01x04") (at 143.51 95.25 0) (unit 1)
+  (symbol (lib_id "Connector_Generic:Conn_01x04") (at 143.51 97.79 0) (mirror x) (unit 1)
     (in_bom yes) (on_board yes) (fields_autoplaced)
-    (property "Reference" "J2" (id 0) (at 145.542 95.6115 0)
-      (effects (font (size 1.27 1.27)) (justify left))
-    )
-    (property "Value" "Conn_01x04" (id 1) (at 145.542 98.3866 0)
-      (effects (font (size 1.27 1.27)) (justify left))
-    )
-    (property "Footprint" "Connector_JST:JST_VH_S4P-VH_1x04_P3.96mm_Horizontal" (id 2) (at 143.51 95.25 0)
+    (property "Reference" "J2" (id 0) (at 143.51 87.4735 0))
+    (property "Value" "Conn_01x04" (id 1) (at 143.51 90.2486 0))
+    (property "Footprint" "Connector_JST:JST_VH_S4P-VH_1x04_P3.96mm_Horizontal" (id 2) (at 143.51 97.79 0)
       (effects (font (size 1.27 1.27)) hide)
     )
-    (property "Datasheet" "~" (id 3) (at 143.51 95.25 0)
+    (property "Datasheet" "~" (id 3) (at 143.51 97.79 0)
       (effects (font (size 1.27 1.27)) hide)
     )
